File: BQ27545.brd (EAGLE design)
At the start: 32.5 x 10 mm, 24 parts, among them U1 Value

Commit message: Add gerber files (exported using elecrow cam job)
Routing:
- net N$2: track 45.4 -> 45.9 mm
Changed lines of the file:
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@@
 <wire x1="29.551" y1="8.06" x2="29.2535" y2="8.06" width="0.3048" layer="1"/>
 <wire x1="29.2535" y1="8.06" x2="29.2535" y2="7.7625" width="0.3048" layer="1"/>
-<wire x1="29.551" y1="8.06" x2="29.551" y2="7.81" width="0.3048" layer="1"/>
-<wire x1="29.551" y1="7.81" x2="30.73" y2="7.81" width="0.3048" layer="1"/>
+<wire x1="30.12" y1="7.81" x2="30.73" y2="7.81" width="0.3048" layer="1"/>
 <wire x1="29.551" y1="8.06" x2="30.73" y2="8.06" width="0.3048" layer="1"/>
 <wire x1="30.73" y1="8.06" x2="30.73" y2="8.572" width="0.3048" layer="1"/>
@@
 <wire x1="29.56" y1="8.2" x2="29.56" y2="7.81" width="0.1524" layer="16"/>
 <wire x1="29.56" y1="7.81" x2="29.206" y2="7.81" width="0.1524" layer="16"/>
-<wire x1="29.551" y1="8.572" x2="29.56" y2="8.572" width="0" layer="19" extent="1-16"/>
+<wire x1="29.551" y1="8.06" x2="29.87" y2="8.06" width="0.1524" layer="1"/>
+<wire x1="29.87" y1="8.06" x2="30.12" y2="7.81" width="0.1524" layer="1"/>
+<wire x1="29.551" y1="8.06" x2="29.551" y2="8.155" width="0.1524" layer="1"/>
+<wire x1="29.551" y1="8.155" x2="29.968" y2="8.572" width="0.1524" layer="1"/>
 </signal>
 <signal name="N$3">
@@
 <mfgpreviewcolor name="substratecolor" color="0xFF786E46"/>
 </mfgpreviewcolors>
+<errors>
+</errors>
 </board>
 </drawing>
